Commit message: insert red color

File: description/robot_core.xacro (robot description, xacro)
@@ -7,4 +7,7 @@
     <material name="orange">
         <color rgba="1 0.3 0.1 1"/>
+    </material>
+    <material name="red">
+        <color rgba="1 0 0 1"/>
     </material>
     <material name="blue">

Commit message: reconfig 2

File: description/robot_core.xacro (robot description, xacro)
@@ -2,4 +2,19 @@
 <robot xmlns:xacro="http://www.ros.org/wiki/xacro" >
     <xacro:include filename="inertial_macros.xacro" />
+    <xacro:property name="chassis_length" value="0.35"/>
+    <xacro:property name="chassis_width" value="0.2"/>
+    <xacro:property name="chassis_height" value="0.16"/>
+    <xacro:property name="chassis_mass" value="0.5"/>
+    <xacro:property name="wheel_radius" value="0.065"/>
+    <xacro:property name="wheel_thickness" value="0.027"/>
+    <xacro:property name="wheel_mass" value="0.1"/>
+    <xacro:property name="wheel_offset_x" value="0.226"/>
+    <xacro:property name="wheel_offset_y" value="0.114"/>
+    <xacro:property name="wheel_offset_z" value="0.01"/>
+    <xacro:property name="chassis_offset_x" value="0.15"/>
+    <xacro:property name="chassis_offset_y" value="0"/>
+    <xacro:property name="chassis_offset_z" value="0.08"/>
+    <xacro:property name="front_offset_x" value="0.155"/>
+    <xacro:property name="back_offset_x" value="0.045"/>
     <material name="white">
         <color rgba="1 1 1 1"/>
@@ -23,4 +38,13 @@
     <link name="base_link">
     </link>
+    <!-- BASE_FOOTPRINT LINK -->
+    <joint name="base_footprint_joint" type="fixed">
+        <parent link="base_link"/>
+        <child link="base_footprint"/>
+        <origin xyz="0 0 0" rpy="0 0 0"/>
+    </joint>
+    <link name="base_footprint">
+    </link>
+    <!--chassy_link-->
     <joint name="chassis_joint" type="fixed">
         <parent link="base_link"/>
@@ -28,21 +52,20 @@
         <origin xyz= "-0.1 0 0"/>
     </joint>
-    <!--chassy_link-->
     <link name="chassis">
         <visual>
-            <origin xyz="0.15 0 0.08"/>
+            <origin xyz="${chassis_offset_x} ${chassis_offset_y} ${chassis_offset_z}"/>
             <geometry>
-                <box size="0.35 0.2 0.13"/>
+                <box size="${chassis_length} ${chassis_width} ${chassis_height}"/>
             </geometry>
             <material name="white"/>
         </visual>
         <collision>
-            <origin xyz="0.15 0 0.08"/>
+            <origin xyz="${chassis_offset_x} ${chassis_offset_y} ${chassis_offset_z}"/>
             <geometry>
-                <box size="0.35 0.2 0.13"/>
+                <box size="${chassis_length} ${chassis_width} ${chassis_height}"/>
             </geometry>
         </collision>
-        <xacro:inertial_box mass="0.5" x="0.35" y="0.2" z="0.13">
-            <origin xyz="0.15 0 0.08" rpy="0 0 0"/>
+        <xacro:inertial_box mass="${chassis_mass}" x="${chassis_length}" y="${chassis_width}" z="${chassis_height}">
+            <origin xyz="${chassis_length/2} 0 ${chassis_height/2}" rpy="0 0 0"/>
         </xacro:inertial_box>
     </link>
@@ -54,5 +77,5 @@
         <parent link="base_link"/>
         <child link="left_front_wheel"/>
-        <origin xyz="0.155 0.114 0" rpy="-${pi/2} 0 0"/>
+        <origin xyz="${front_offset_x} ${wheel_offset_y} 0" rpy="-${pi/2} 0 0"/>
         <axis xyz="0 0 1"/>
     </joint>
@@ -60,5 +83,5 @@
         <visual>
             <geometry>
-                <cylinder radius="0.065" length="0.027"/>
+                <cylinder radius="${wheel_radius}" length="${wheel_thickness}"/>
             </geometry>
             <material name="blue"/>
@@ -66,8 +89,8 @@
         <collision>
             <geometry>
-                <cylinder radius="0.065" length="0.027"/>
+                <cylinder radius="${wheel_radius}" length="${wheel_thickness}"/>
             </geometry>
         </collision>
-            <xacro:inertial_cylinder mass="0.1" length="0.027" radius="0.065">
+            <xacro:inertial_cylinder mass="${wheel_mass}" length="${wheel_thickness}" radius="${wheel_radius}">
                 <origin xyz="0 0 0" rpy="0 0 0"/>
             </xacro:inertial_cylinder>
@@ -80,5 +103,5 @@
         <parent link="base_link"/>
         <child link="right_front_wheel"/>
-        <origin xyz="0.155 -0.114 0" rpy="${pi/2} 0 0"/>
+        <origin xyz="${front_offset_x} ${-wheel_offset_y} 0" rpy="${pi/2} 0 0"/>
         <axis xyz="0 0 -1"/>
     </joint>
@@ -86,5 +109,5 @@
         <visual>
             <geometry>
-                <cylinder radius="0.065" length="0.027"/>
+                <cylinder radius="${wheel_radius}" length="${wheel_thickness}"/>
             </geometry>
             <material name="blue"/>
@@ -92,8 +115,8 @@
         <collision>
             <geometry>
-                <cylinder radius="0.065" length="0.027"/>
+                <cylinder radius="${wheel_radius}" length="${wheel_thickness}"/>
             </geometry>
         </collision>
-            <xacro:inertial_cylinder mass="0.1" length="0.027" radius="0.065">
+            <xacro:inertial_cylinder mass="${wheel_mass}" length="${wheel_thickness}" radius="${wheel_radius}">
                 <origin xyz="0 0 0" rpy="0 0 0"/>
             </xacro:inertial_cylinder>
@@ -106,5 +129,5 @@
         <parent link="base_link"/>
         <child link="left_back_wheel"/>
-        <origin xyz="-0.045 0.114 0" rpy="-${pi/2} 0 0"/>
+        <origin xyz="${-back_offset_x} ${wheel_offset_y} 0" rpy="-${pi/2} 0 0"/>
         <axis xyz="0 0 1"/>
     </joint>
@@ -112,5 +135,5 @@
         <visual>
             <geometry>
-                <cylinder radius="0.065" length="0.027"/>
+                <cylinder radius="${wheel_radius}" length="${wheel_thickness}"/>
             </geometry>
             <material name="blue"/>
@@ -118,8 +141,8 @@
         <collision>
             <geometry>
-                <cylinder radius="0.065" length="0.027"/>
+                <cylinder radius="${wheel_radius}" length="${wheel_thickness}"/>
             </geometry>
         </collision>
-            <xacro:inertial_cylinder mass="0.1" length="0.027" radius="0.065">
+            <xacro:inertial_cylinder mass="${wheel_mass}" length="${wheel_thickness}" radius="${wheel_radius}">
                 <origin xyz="0 0 0" rpy="0 0 0"/>
             </xacro:inertial_cylinder>
@@ -132,5 +155,5 @@
         <parent link="base_link"/>
         <child link="right_back_wheel"/>
-        <origin xyz="-0.045 -0.114 0" rpy="${pi/2} 0 0"/>
+        <origin xyz="${-back_offset_x} ${-wheel_offset_y} 0" rpy="${pi/2} 0 0"/>
         <axis xyz="0 0 -1"/>
     </joint>
@@ -138,5 +161,5 @@
         <visual>
             <geometry>
-                <cylinder radius="0.065" length="0.027"/>
+                <cylinder radius="${wheel_radius}" length="${wheel_thickness}"/>
             </geometry>
             <material name="blue"/>
@@ -144,8 +167,8 @@
         <collision>
             <geometry>
-                <cylinder radius="0.065" length="0.027"/>
+                <cylinder radius="${wheel_radius}" length="${wheel_thickness}"/>
             </geometry>
         </collision>
-            <xacro:inertial_cylinder mass="0.1" length="0.027" radius="0.065">
+            <xacro:inertial_cylinder mass="${wheel_mass}" length="${wheel_thickness}" radius="${wheel_radius}">
                 <origin xyz="0 0 0" rpy="0 0 0"/>
             </xacro:inertial_cylinder>
